File: mainboard.kicad_pcb (KiCad board)
At the start: 2 copper layers, 108 x 48.3 mm, 108 parts, among them IC1 LM4558N, IC2 LM4558N, IC3 LM4558N

Commit message: pisc
Other:
- board text added: "npn: bc547 pnp: bc557"
Changed lines of the file:
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@@
+		)
+	)
+	(gr_text "npn: bc547\npnp: bc557"
+		(at 100 121 90)
+		(layer "F.SilkS")
+		(effects
+			(font
+				(size 1.5 1.5)
+				(thickness 0.3)
+				(bold yes)
+			)
+			(justify left bottom)
 		)
 	)

Commit message: asd
Parts:
- T1, T10, T11, T12, T13, T14, T16, T18, T19, T20, T3, T5, T6, T8: value (none) -> BC547
- T15, T17, T2, T4, T7, T9: value (none) -> BC557B
Changed lines of the file:
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@@
 			)
 		)
-		(property "Value" ""
+		(property "Value" "BC547"
 			(at -2.54 3.302 90)
 			(unlocked yes)
@@
 			)
 		)
-		(property "Value" ""
+		(property "Value" "BC557B"
 			(at -2.54 4.572 90)
 			(unlocked yes)
@@
 			)
 		)
-		(property "Footprint" ""
+		(property "Footprint" "mainboard:TO92-EBC"
 			(at 0 0 90)
 			(layer "F.Fab")
@@
 			)
 		)
-		(property "Value" ""
+		(property "Value" "BC557B"
 			(at -2.54 4.572 0)
 			(unlocked yes)
@@
 			)
 		)
-		(property "Footprint" ""
+		(property "Footprint" "mainboard:TO92-EBC"
 			(at 0 0 180)
 			(layer "F.Fab")
@@
 			)
 		)
-		(property "Value" ""
+		(property "Value" "BC547"
 			(at -2.54 3.302 90)
 			(unlocked yes)
@@
 			)
 		)
-		(property "Value" ""
+		(property "Value" "BC547"
 			(at -2.54 3.302 90)
 			(unlocked yes)
@@
 			)
 		)
-		(property "Value" ""
+		(property "Value" "BC547"
 			(at -2.54 3.302 0)
 			(unlocked yes)
@@
 			)
 		)
-		(property "Value" ""
+		(property "Value" "BC547"
 			(at -2.54 3.302 90)
 			(unlocked yes)
@@
 		)
 		(property "Footprint" ""
-			(at 0 0 -90)
+			(at 0 0 90)
 			(layer "F.Fab")
 			(hide yes)
@@
 		)
 		(property "Datasheet" ""
-			(at 0 0 -90)
+			(at 0 0 90)
 			(layer "F.Fab")
 			(hide yes)
@@
 		)
 		(property "Description" ""
-			(at 0 0 -90)
+			(at 0 0 90)
 			(layer "F.Fab")
 			(hide yes)
@@
 			)
 		)
-		(property "Value" ""
+		(property "Value" "BC547"
 			(at -2.54 3.302 0)
 			(unlocked yes)
@@
 			)
 		)
-		(property "Value" ""
+		(property "Value" "BC547"
 			(at -2.54 3.302 90)
 			(unlocked yes)
@@
 			)
 		)
-		(property "Value" ""
+		(property "Value" "BC547"
 			(at -2.54 3.302 90)
 			(unlocked yes)
@@
 			)
 		)
-		(property "Value" ""
+		(property "Value" "BC547"
 			(at -2.54 3.302 90)
 			(unlocked yes)
@@
 			)
 		)
-		(property "Value" ""
+		(property "Value" "BC557B"
 			(at -2.54 4.572 90)
 			(unlocked yes)
@@
 			)
 		)
-		(property "Footprint" ""
-			(at 0 0 -90)
+		(property "Footprint" "mainboard:TO92-EBC"
+			(at 0 0 90)
 			(layer "F.Fab")
 			(hide yes)
@@
 		)
 		(property "Datasheet" ""
-			(at 0 0 -90)
+			(at 0 0 90)
 			(layer "F.Fab")
 			(hide yes)
@@
 		)
 		(property "Description" ""
-			(at 0 0 -90)
+			(at 0 0 90)
 			(layer "F.Fab")
 			(hide yes)
@@
 			)
 		)
-		(property "Value" ""
+		(property "Value" "BC547"
 			(at -2.54 3.302 90)
 			(unlocked yes)
@@
 		)
 		(property "Footprint" ""
-			(at 0 0 -90)
+			(at 0 0 90)
 			(layer "F.Fab")
 			(hide yes)
@@
 		)
 		(property "Datasheet" ""
-			(at 0 0 -90)
+			(at 0 0 90)
 			(layer "F.Fab")
 			(hide yes)
@@
 		)
 		(property "Description" ""
-			(at 0 0 -90)
+			(at 0 0 90)
 			(layer "F.Fab")
 			(hide yes)
@@
 			)
 		)
-		(property "Value" ""
+		(property "Value" "BC547"
 			(at -2.54 3.302 0)
 			(unlocked yes)
@@
 			)
 		)
-		(property "Value" ""
+		(property "Value" "BC557B"
 			(at -2.54 4.572 0)
 			(unlocked yes)
@@
 			)
 		)
-		(property "Footprint" ""
+		(property "Footprint" "mainboard:TO92-EBC"
 			(at 0 0 0)
 			(layer "F.Fab")
@@
 			)
 		)
-		(property "Value" ""
+		(property "Value" "BC547"
 			(at -2.54 3.302 90)
 			(unlocked yes)
@@
 		)
 		(property "Footprint" ""
-			(at 0 0 -90)
+			(at 0 0 90)
 			(layer "F.Fab")
 			(hide yes)
@@
 		)
 		(property "Datasheet" ""
-			(at 0 0 -90)
+			(at 0 0 90)
 			(layer "F.Fab")
 			(hide yes)
@@
 		)
 		(property "Description" ""
-			(at 0 0 -90)
+			(at 0 0 90)
 			(layer "F.Fab")
 			(hide yes)
@@
 			)
 		)
-		(property "Value" ""
+		(property "Value" "BC557B"
 			(at -2.54 4.572 90)
 			(unlocked yes)
@@
 			)
 		)
-		(property "Footprint" ""
-			(at 0 0 -90)
+		(property "Footprint" "mainboard:TO92-EBC"
+			(at 0 0 90)
 			(layer "F.Fab")
 			(hide yes)
@@
 		)
 		(property "Datasheet" ""
-			(at 0 0 -90)
+			(at 0 0 90)
 			(layer "F.Fab")
 			(hide yes)
@@
 		)
 		(property "Description" ""
-			(at 0 0 -90)
+			(at 0 0 90)
 			(layer "F.Fab")
 			(hide yes)
@@
 			)
 		)
-		(property "Value" ""
+		(property "Value" "BC557B"
 			(at -2.54 4.572 90)
 			(unlocked yes)
@@
 			)
 		)
-		(property "Footprint" ""
+		(property "Footprint" "mainboard:TO92-EBC"
 			(at 0 0 90)
 			(layer "F.Fab")
@@
 			)
 		)
-		(property "Value" ""
+		(property "Value" "BC547"
 			(at -2.54 3.302 90)
 			(unlocked yes)
@@
 		)
 		(property "Footprint" ""
-			(at 0 0 -90)
+			(at 0 0 90)
 			(layer "F.Fab")
 			(hide yes)
@@
 		)
 		(property "Datasheet" ""
-			(at 0 0 -90)
+			(at 0 0 90)
 			(layer "F.Fab")
 			(hide yes)
@@
 		)
 		(property "Description" ""
-			(at 0 0 -90)
+			(at 0 0 90)
 			(layer "F.Fab")
 			(hide yes)
@@
 			)
 		)
-		(property "Value" ""
+		(property "Value" "BC547"
 			(at -2.54 3.302 90)
 			(unlocked yes)
@@
 		)
 		(property "Footprint" ""
-			(at 0 0 -90)
+			(at 0 0 90)
 			(layer "F.Fab")
 			(hide yes)
@@
 		)
 		(property "Datasheet" ""
-			(at 0 0 -90)
+			(at 0 0 90)
 			(layer "F.Fab")
 			(hide yes)
@@
 		)
 		(property "Description" ""
-			(at 0 0 -90)
+			(at 0 0 90)
 			(layer "F.Fab")
 			(hide yes)
