File: mainboard.kicad_sch (KiCad schematic)
At the start: 104 parts, among them IC1 4558N, IC2 4558N, IC3 4558N, T1 -NPN-TO92-CBE, T10 -NPN-TO92-CBE, T11 -NPN-TO92-CBE, T12 -NPN-TO92-CBE, T13 -NPN-TO92-CBE, T14 -NPN-TO92-CBE, T15 -PNP-TO92-EBC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

Commit message: pisc
Parts:
- T1, T10, T11, T12, T13, T14, T16, T18, T19, T20, T3, T5, T6, T8: value -NPN-TO92-CBE -> BC547B-NPN-CBE
- T15, T17, T2, T4, T7, T9: value -PNP-TO92-EBC -> BC557B-PNP-EBC
Changed lines of the file:
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@@
 			)
 		)
-		(property "Value" "-NPN-TO92-CBE"
+		(property "Value" "BC547B-NPN-CBE"
 			(at 322.58 322.58 0)
 			(effects
@@
 			)
 		)
-		(property "Value" "-PNP-TO92-EBC"
+		(property "Value" "BC557B-PNP-EBC"
 			(at 396.24 317.5 0)
 			(effects
@@
 			)
 		)
-		(property "Value" "-NPN-TO92-CBE"
+		(property "Value" "BC547B-NPN-CBE"
 			(at 381 350.52 0)
 			(effects
@@
 			)
 		)
-		(property "Value" "-NPN-TO92-CBE"
+		(property "Value" "BC547B-NPN-CBE"
 			(at 396.24 292.1 0)
 			(effects
@@
 			)
 		)
-		(property "Value" "-NPN-TO92-CBE"
+		(property "Value" "BC547B-NPN-CBE"
 			(at 347.98 218.44 0)
 			(effects
@@
 			)
 		)
-		(property "Value" "-PNP-TO92-EBC"
+		(property "Value" "BC557B-PNP-EBC"
 			(at 208.28 157.48 0)
 			(effects
@@
 			)
 		)
-		(property "Value" "-PNP-TO92-EBC"
+		(property "Value" "BC557B-PNP-EBC"
 			(at 114.3 68.58 0)
 			(effects
@@
 			)
 		)
-		(property "Value" "-NPN-TO92-CBE"
+		(property "Value" "BC547B-NPN-CBE"
 			(at 193.04 190.5 0)
 			(effects
@@
 			)
 		)
-		(property "Value" "-PNP-TO92-EBC"
+		(property "Value" "BC557B-PNP-EBC"
 			(at 393.7 243.84 0)
 			(effects
@@
 			)
 		)
-		(property "Value" "-NPN-TO92-CBE"
+		(property "Value" "BC547B-NPN-CBE"
 			(at 208.28 132.08 0)
 			(effects
@@
 			)
 		)
-		(property "Value" "-NPN-TO92-CBE"
+		(property "Value" "BC547B-NPN-CBE"
 			(at 134.62 162.56 0)
 			(effects
@@
 			)
 		)
-		(property "Value" "-NPN-TO92-CBE"
+		(property "Value" "BC547B-NPN-CBE"
 			(at 370.84 358.14 0)
 			(effects
@@
 			)
 		)
-		(property "Value" "-NPN-TO92-CBE"
+		(property "Value" "BC547B-NPN-CBE"
 			(at 198.12 149.86 0)
 			(effects
@@
 			)
 		)
-		(property "Value" "-NPN-TO92-CBE"
+		(property "Value" "BC547B-NPN-CBE"
 			(at 281.94 236.22 0)
 			(effects
@@
 			)
 		)
-		(property "Value" "-NPN-TO92-CBE"
+		(property "Value" "BC547B-NPN-CBE"
 			(at 386.08 309.88 0)
 			(effects
@@
 			)
 		)
-		(property "Value" "-NPN-TO92-CBE"
+		(property "Value" "BC547B-NPN-CBE"
 			(at 160.02 58.42 0)
 			(effects
@@
 			)
 		)
-		(property "Value" "-PNP-TO92-EBC"
+		(property "Value" "BC557B-PNP-EBC"
 			(at 205.74 83.82 0)
 			(effects
@@
 			)
 		)
-		(property "Value" "-NPN-TO92-CBE"
+		(property "Value" "BC547B-NPN-CBE"
 			(at 93.98 76.2 0)
 			(effects
@@
 			)
 		)
-		(property "Value" "-PNP-TO92-EBC"
+		(property "Value" "BC557B-PNP-EBC"
 			(at 302.26 228.6 0)
 			(effects
@@
 			)
 		)
-		(property "Value" "-NPN-TO92-CBE"
+		(property "Value" "BC547B-NPN-CBE"
 			(at 182.88 198.12 0)
 			(effects
